Commit message: added a dummy base for urdf, to align with real robot coordinate system

File: colcon_ws/src/duco_gcr5_910_urdf/urdf/duco_gcr5_910_urdf.urdf (robot description, URDF)
Before this commit: robot duco_gcr5_910_urdf, 7 links, 6 joints
Links:
- added link rotated_base
Joints:
- added joint base_rotation: type fixed, parent rotated_base, child base_link, origin xyz=0 0 0 rpy=0 0 -1.5708
- joint joint1: axis -1 0 0 -> 1 0 0
- joint joint2: axis -1 0 0 -> 1 0 0
- joint joint3: axis -1 0 0 -> 1 0 0
- joint joint5: axis 0 0 1 -> 0 0 -1

Commit message: fixed urdf model error, previously the assembly was wrong

File: colcon_ws/src/duco_gcr5_910_urdf/urdf/duco_gcr5_910_urdf.urdf (robot description, URDF)
Before this commit: robot duco_gcr5_910_urdf, 8 links, 7 joints
Links:
- link link1: mass 0.424385093655344 -> 0.424385142287687
- link link2: mass 1.1009274409569 -> 1.10092744951388
- link link3: mass 0.330047321805258 -> 0.330047308889306
- link link4: mass 0.165023508277068 -> 0.165024183426076
- link link5: mass 0.148290193529033 -> 0.148289061509009
- link link6: mass 0.270719809445498 -> 0.270719809172517
Joints:
- joint joint2: origin xyz=0.122 0.0052441786897741 0 rpy=3.14159265358979 0 1.5707963267949 -> xyz=0.122 0.00524417868977412 0 rpy=-3.14159265358979 0 1.5707963267949
- joint joint4: axis 0 -1 0 -> 1 0 0; origin xyz=0.018076 0.392 0 rpy=3.1416 0 -1.5708 -> xyz=0.00701337927126169 0.391999999998075 0 rpy=0 0 0
- joint joint5: origin xyz=-0.0027576 -0.08618 0 rpy=3.1416 -1.5708 0 -> xyz=0.128242442033315 0 0 rpy=1.5707963267949 1.5707963267949 0
- joint joint6: origin xyz=0 0.047999999999999 -0.128242442033315 rpy=0 0 -3.14159265358979 -> xyz=0 0.0480000000046998 -0.0999999999991573 rpy=0 0 -3.14159265358979
