Commit message: Refactor: Clean up legacy packages and migrate to official ROS2 Control
- Remove obsolete duco_arms package (dual-arm config not needed)
- Simplify duco_ros_driver to library-only package (remove executable nodes with duco_msg dependencies)
- Update package dependencies to remove references to deleted duco_msg and duco_arms
- Fix launch file parameter passing for robot_ip and robot_port configuration
- Update README.md with current package structure and VMware deployment guide
- Maintain backward compatibility for hardware interface and mesh files

This commit completes the migration to official ROS2 Control architecture while removing deprecated custom message packages.

File: colcon_ws/src/duco_gcr5_910_moveit_config/config/gcr5_910.ros2_control.xacro (robot description, xacro)
@@ -1,12 +1,12 @@
 <?xml version="1.0"?>
 <robot xmlns:xacro="http://www.ros.org/wiki/xacro">
-    <xacro:macro name="gcr5_910_ros2_control" params="name initial_positions_file">
-        <xacro:property name="initial_positions" value="${load_yaml(initial_positions_file)['initial_positions']}"/>
+    <xacro:macro name="gcr5_910_ros2_control" params="name initial_positions_file robot_ip:=192.168.1.10 robot_port:=7003">
+        <xacro:property name="initial_positions" value="${xacro.load_yaml(initial_positions_file)['initial_positions']}"/>
         <ros2_control name="${name}" type="system">
             <hardware>
                 <!-- Real DUCO hardware interface -->
                 <plugin>duco_hardware/DucoHardwareInterface</plugin>
-                <param name="robot_ip">192.168.1.10</param>
-                <param name="robot_port">7003</param>
+                <param name="robot_ip">${robot_ip}</param>
+                <param name="robot_port">${robot_port}</param>
             </hardware>
             <joint name="arm_1_joint_1">

File: colcon_ws/src/duco_gcr5_910_moveit_config/config/gcr5_910.urdf.xacro (robot description, xacro)
@@ -2,8 +2,10 @@
 <robot xmlns:xacro="http://www.ros.org/wiki/xacro" name="gcr5_910">
     <xacro:arg name="initial_positions_file" default="initial_positions.yaml" />
+    <xacro:arg name="robot_ip" default="192.168.1.10" />
+    <xacro:arg name="robot_port" default="7003" />
     <!-- Import gcr5_910 urdf file -->
     <xacro:include filename="$(find duco_support)/urdf/duco_gcr5_910.urdf" />
     <!-- Import control_xacro -->
     <xacro:include filename="gcr5_910.ros2_control.xacro" />
-    <xacro:gcr5_910_ros2_control name="FakeSystem" initial_positions_file="$(arg initial_positions_file)"/>
+    <xacro:gcr5_910_ros2_control name="FakeSystem" initial_positions_file="$(arg initial_positions_file)" robot_ip="$(arg robot_ip)" robot_port="$(arg robot_port)"/>
 </robot>
